Commit message: [update] new assets

File: resources/models/environment_assets/trees/tree_0.urdf (robot description, URDF)
Before this commit: robot tree_0.urdf, 13 links, 12 joints
Links:
- link branch_1: mass 1.0 -> 0.0
- link branch_10: mass 1.0 -> 0.0
- link branch_11: mass 1.0 -> 0.0
- link branch_12: mass 1.0 -> 0.0
- link branch_2: mass 1.0 -> 0.0
- link branch_3: mass 1.0 -> 0.0
- link branch_4: mass 1.0 -> 0.0
- link branch_5: mass 1.0 -> 0.0
- link branch_6: mass 1.0 -> 0.0
- link branch_7: mass 1.0 -> 0.0
- link branch_8: mass 1.0 -> 0.0
- link branch_9: mass 1.0 -> 0.0

File: resources/models/environment_assets/trees/tree_1.urdf (robot description, URDF)
Before this commit: robot tree_1.urdf, 13 links, 12 joints
Links:
- link branch_1: mass 1.0 -> 0.0
- link branch_10: mass 1.0 -> 0.0
- link branch_11: mass 1.0 -> 0.0
- link branch_12: mass 1.0 -> 0.0
- link branch_2: mass 1.0 -> 0.0
- link branch_3: mass 1.0 -> 0.0
- link branch_4: mass 1.0 -> 0.0
- link branch_5: mass 1.0 -> 0.0
- link branch_6: mass 1.0 -> 0.0
- link branch_7: mass 1.0 -> 0.0
- link branch_8: mass 1.0 -> 0.0
- link branch_9: mass 1.0 -> 0.0
