Commit message: [add] ground as asset

File: resources/models/environment_assets/boundaries/8X18ground/model.urdf (robot description, URDF)
Before this commit: robot 18X8ground, 1 links, 0 joints
Links:
- link base_link: geometry collision mesh filename=8X18ground.dae scale=1. 1. 1.; visual mesh filename=8X18ground.dae scale=1. 1. 1.

File: resources/models/environment_assets/boundaries/8X8ground/model.urdf (robot description, URDF)
Before this commit: robot 18X18ground, 1 links, 0 joints
Links:
- link base_link: geometry collision mesh filename=8X8ground.dae scale=1. 1. 1.; visual mesh filename=8X8ground.dae scale=1. 1. 1.
