Commit message: [update] atti nn model

File: resources/robots/X152b/model.urdf (robot description, URDF)
Before this commit: robot quadrotor, 5 links, 4 joints
Links:
- link base_link: mass 0.58 -> 0.295

Commit message: [update] asset manager

File: resources/robots/X152b/model.urdf (robot description, URDF)
Before this commit: robot quadrotor, 5 links, 4 joints
Links:
- link base_link: mass 0.295 -> 0.58

Commit message: [test]

File: resources/robots/X152b/model.urdf (robot description, URDF)
Before this commit: robot quadrotor, 5 links, 4 joints
Links:
- link base_link: mass 0.58 -> 0.585
