Commit message: [fix] 1X1cube

File: resources/models/environment_assets/cubes/1X1/model.urdf (robot description, URDF)
Before this commit: robot 1x1cube, 1 links, 0 joints
Links:
- link base_link: geometry collision mesh filename=1x1dae.dae scale=1. 1. 1.; visual mesh filename=1x1dae.dae scale=1. 1. 1.
