Commit message: [update]

File: resources/models/environment_assets/balls/balloon/model.urdf (robot description, URDF)
Before this commit: robot ellipsoid, 1 links, 0 joints
Links:
- link ellipsoid: geometry collision mesh filename=ellipsoid_balloon.stl scale=.2 .2 .2; visual mesh filename=ellipsoid_balloon.stl scale=.2 .2 .2
