Commit message: [add] new task planning

File: resources/models/environment_assets/thin/tree_0.urdf (robot description, URDF)
Before this commit: robot tree_0.urdf, 1 links, 0 joints
Links:
- link branch_0: geometry collision cylinder length=2.426672438829133 radius=0.05609708829281466; visual cylinder length=2.426672438829133 radius=0.05609708829281466

File: resources/models/environment_assets/thin/tree_1.urdf (robot description, URDF)
Before this commit: robot tree_1.urdf, 1 links, 0 joints
Links:
- link branch_0: geometry collision cylinder length=3.4570259582678617 radius=0.04038201981897694; visual cylinder length=3.4570259582678617 radius=0.04038201981897694

File: resources/models/environment_assets/thin/tree_10.urdf (robot description, URDF)
Before this commit: robot tree_10.urdf, 1 links, 0 joints
Links:
- link branch_0: geometry collision cylinder length=2.8787618557428076 radius=0.06959517276692666; visual cylinder length=2.8787618557428076 radius=0.06959517276692666

File: resources/models/environment_assets/thin/tree_11.urdf (robot description, URDF)
Before this commit: robot tree_11.urdf, 1 links, 0 joints
Links:
- link branch_0: geometry collision cylinder length=3.457460186809768 radius=0.032937656047029557; visual cylinder length=3.457460186809768 radius=0.032937656047029557

File: resources/models/environment_assets/thin/tree_12.urdf (robot description, URDF)
Before this commit: robot tree_12.urdf, 1 links, 0 joints
Links:
- link branch_0: geometry collision cylinder length=3.754936539643756 radius=0.03322757579081633; visual cylinder length=3.754936539643756 radius=0.03322757579081633

File: resources/models/environment_assets/thin/tree_13.urdf (robot description, URDF)
Before this commit: robot tree_13.urdf, 1 links, 0 joints
Links:
- link branch_0: geometry collision cylinder length=2.2322939761545797 radius=0.03091524220594921; visual cylinder length=2.2322939761545797 radius=0.03091524220594921

File: resources/models/environment_assets/thin/tree_14.urdf (robot description, URDF)
Before this commit: robot tree_14.urdf, 1 links, 0 joints
Links:
- link branch_0: geometry collision cylinder length=2.5262356605409977 radius=0.06623314568882309; visual cylinder length=2.5262356605409977 radius=0.06623314568882309

File: resources/models/environment_assets/thin/tree_15.urdf (robot description, URDF)
Before this commit: robot tree_15.urdf, 1 links, 0 joints
Links:
- link branch_0: geometry collision cylinder length=2.5327326848287033 radius=0.05221642493124601; visual cylinder length=2.5327326848287033 radius=0.05221642493124601

File: resources/models/environment_assets/thin/tree_16.urdf (robot description, URDF)
Before this commit: robot tree_16.urdf, 1 links, 0 joints
Links:
- link branch_0: geometry collision cylinder length=2.632392683107045 radius=0.048564732780250267; visual cylinder length=2.632392683107045 radius=0.048564732780250267

File: resources/models/environment_assets/thin/tree_17.urdf (robot description, URDF)
Before this commit: robot tree_17.urdf, 1 links, 0 joints
Links:
- link branch_0: geometry collision cylinder length=2.2238522360668496 radius=0.037459574625546985; visual cylinder length=2.2238522360668496 radius=0.037459574625546985

File: resources/models/environment_assets/thin/tree_18.urdf (robot description, URDF)
Before this commit: robot tree_18.urdf, 1 links, 0 joints
Links:
- link branch_0: geometry collision cylinder length=2.4151181239384094 radius=0.05755079824530901; visual cylinder length=2.4151181239384094 radius=0.05755079824530901

File: resources/models/environment_assets/thin/tree_19.urdf (robot description, URDF)
Before this commit: robot tree_19.urdf, 1 links, 0 joints
Links:
- link branch_0: geometry collision cylinder length=3.982587941395516 radius=0.03936485466384738; visual cylinder length=3.982587941395516 radius=0.03936485466384738

File: resources/models/environment_assets/thin/tree_2.urdf (robot description, URDF)
Before this commit: robot tree_2.urdf, 1 links, 0 joints
Links:
- link branch_0: geometry collision cylinder length=3.188981571307792 radius=0.07190169378059089; visual cylinder length=3.188981571307792 radius=0.07190169378059089

File: resources/models/environment_assets/thin/tree_20.urdf (robot description, URDF)
Before this commit: robot tree_20.urdf, 1 links, 0 joints
Links:
- link branch_0: geometry collision cylinder length=3.337894987637521 radius=0.06293721026315051; visual cylinder length=3.337894987637521 radius=0.06293721026315051

File: resources/models/environment_assets/thin/tree_21.urdf (robot description, URDF)
Before this commit: robot tree_21.urdf, 1 links, 0 joints
Links:
- link branch_0: geometry collision cylinder length=2.0843962251670916 radius=0.04788944814374537; visual cylinder length=2.0843962251670916 radius=0.04788944814374537

File: resources/models/environment_assets/thin/tree_22.urdf (robot description, URDF)
Before this commit: robot tree_22.urdf, 1 links, 0 joints
Links:
- link branch_0: geometry collision cylinder length=3.3361616993822953 radius=0.07082931836432933; visual cylinder length=3.3361616993822953 radius=0.07082931836432933

File: resources/models/environment_assets/thin/tree_23.urdf (robot description, URDF)
Before this commit: robot tree_23.urdf, 1 links, 0 joints
Links:
- link branch_0: geometry collision cylinder length=3.3667963991007057 radius=0.057918416088893074; visual cylinder length=3.3667963991007057 radius=0.057918416088893074

File: resources/models/environment_assets/thin/tree_24.urdf (robot description, URDF)
Before this commit: robot tree_24.urdf, 1 links, 0 joints
Links:
- link branch_0: geometry collision cylinder length=3.1099634793560997 radius=0.06664560730124382; visual cylinder length=3.1099634793560997 radius=0.06664560730124382

File: resources/models/environment_assets/thin/tree_25.urdf (robot description, URDF)
Before this commit: robot tree_25.urdf, 1 links, 0 joints
Links:
- link branch_0: geometry collision cylinder length=3.3265214117656146 radius=0.043011255719930745; visual cylinder length=3.3265214117656146 radius=0.043011255719930745

File: resources/models/environment_assets/thin/tree_26.urdf (robot description, URDF)
Before this commit: robot tree_26.urdf, 1 links, 0 joints
Links:
- link branch_0: geometry collision cylinder length=2.2891687826951927 radius=0.048793203332612965; visual cylinder length=2.2891687826951927 radius=0.048793203332612965
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