Commit message: [add] vae encoding

File: airgym/assets/env_assets/objects/cube.urdf (robot description, URDF)
Before this commit: robot box, 1 links, 0 joints
Links:
- link base_link: geometry collision box size=.6 .6 .6; visual box size=.6 .6 .6

File: airgym/assets/env_assets/objects/cuboidal_rod.urdf (robot description, URDF)
Before this commit: robot box, 1 links, 0 joints
Links:
- link base_link: geometry collision box size=0.15 0.15 1.0; visual box size=0.15 0.15 1.0
